File: showdown_gun_board.kicad_pcb (KiCad board)
At the start: 2 copper layers, 31 parts, among them J1 Conn_01x04_Pin, J2 USB4155-03-C_REVA, SW1 SW_SPDT, U1 AMS1117-3.3, U2 MCP6002-xMC, U3 STM32F103C8T6, Y1 16MHz

Commit message: null
Parts:
- removed C1, C2: 22uF, Capacitor_SMD:C_0603_1608Metric
- removed C10, C4, C6, C8, C9: 100nF, Capacitor_SMD:C_0603_1608Metric
- removed C11: 10nF, Capacitor_SMD:C_0603_1608Metric
- removed C12, C13: 1uF, Capacitor_SMD:C_0603_1608Metric
- removed C3: 10uF, Capacitor_SMD:C_0603_1608Metric
- removed C5, C7: 10pF, Capacitor_SMD:C_0603_1608Metric
- removed D1: BPX65, Package_TO_SOT_THT:TO-18-2_Lens
- removed D2: LED_RED, LED_SMD:LED_0805_2012Metric
- removed FB1: 120R, Inductor_SMD:L_0603_1608Metric
- removed J1: Conn_01x04_Pin, Connector_PinHeader_2.54mm:PinHeader_1x04_P2.54mm_Horizontal
- removed J2: USB4155-03-C_REVA, USB4155-03-C_REVA:GCT_USB4155-03-C_REVA
- removed R1, R2, R3, R5: 1.5K, Resistor_SMD:R_0603_1608Metric
- removed R1, R7: 1M, Resistor_SMD:R_0603_1608Metric
- removed R4: 10K, Resistor_SMD:R_0603_1608Metric
- removed R6: 5.1K, Resistor_SMD:R_0603_1608Metric
- removed SW1: SW_SPDT, Button_Switch_THT:SW_E-Switch_EG1271_SPDT
- removed U1: AMS1117-3.3, Package_TO_SOT_SMD:SOT-223-3_TabPin2
- removed U3: STM32F103C8T6, Package_QFP:LQFP-48_7x7mm_P0.5mm
- removed Y1: 16MHz, Crystal:Crystal_SMD_3225-4Pin_3.2x2.5mm
- added C14: 22uF, Capacitor_SMD:C_0603_1608Metric, F.Cu at (126.4, 97.5)
- added C15: 22uF, Capacitor_SMD:C_0603_1608Metric, F.Cu at (126.4, 100.0)
- added C16: 10uF, Capacitor_SMD:C_0603_1608Metric, F.Cu at (126.4, 102.5)
- added C17: 100nF, Capacitor_SMD:C_0603_1608Metric, F.Cu at (126.4, 105.0)
- added C18: 10pF, Capacitor_SMD:C_0603_1608Metric, F.Cu at (126.4, 107.5)
- added C19: 100nF, Capacitor_SMD:C_0603_1608Metric, F.Cu at (126.4, 110.0)
- added C20: 10pF, Capacitor_SMD:C_0603_1608Metric, F.Cu at (130.5, 97.5)
- added C22: 100nF, Capacitor_SMD:C_0603_1608Metric, F.Cu at (130.5, 100.0)
- added C23: 100nF, Capacitor_SMD:C_0603_1608Metric, F.Cu at (130.5, 102.5)
- added C24: 100nF, Capacitor_SMD:C_0603_1608Metric, F.Cu at (130.5, 105.0)
- added C25: 10nF, Capacitor_SMD:C_0603_1608Metric, F.Cu at (130.5, 107.5)
- added C26: 1uF, Capacitor_SMD:C_0603_1608Metric, F.Cu at (130.5, 110.0)
- added C27: 1uF, Capacitor_SMD:C_0603_1608Metric, F.Cu at (134.5, 97.5)
- added D4: LED_RED, LED_SMD:LED_0805_2012Metric, F.Cu at (148.6, 110.0)
- added FB2: 120R, Inductor_SMD:L_0603_1608Metric, F.Cu at (134.5, 100.0)
- added J3: USB_B_Micro, Connector_USB:USB_Micro-AB_Molex_47590-0001, F.Cu at (142.2, 100.9)
- added J4: Conn_01x04_Pin, Connector_PinHeader_2.54mm:PinHeader_1x04_P2.54mm_Horizontal, F.Cu at (126.8, 86.3)
- added R18: 1.5K, Resistor_SMD:R_0603_1608Metric, F.Cu at (134.5, 102.5)
- added R19: 10K, Resistor_SMD:R_0603_1608Metric, F.Cu at (134.5, 105.0)
- added R21: 1.5K, Resistor_SMD:R_0603_1608Metric, F.Cu at (134.5, 107.5)
- added SW2: SW_SPDT, Button_Switch_THT:SW_Slide-03_Wuerth-WS-SLTV_10x2.5x6.4_P2.54mm, F.Cu at (130.2, 113.3)
- added U6: STM32F103C8T6, Package_QFP:LQFP-48_7x7mm_P0.5mm, F.Cu at (143.5, 89.6)
- added Y2: 16MHz, Crystal:Crystal_SMD_3225-4Pin_3.2x2.5mm, F.Cu at (148.9, 106.3)
- U2: value MCP6002-xMC -> AMS1117-3.3; footprint Package_DFN_QFN:DFN-8-1EP_3x2mm_P0.5mm_EP1.75x1.45mm -> Package_TO_SOT_SMD:SOT-223-3_TabPin2
- moved U2 38.7 mm to (141.4, 108.2)
Connections:
- U2 pad 1: /hit_register -> GND
- U2 pad 2: Net-(U2A--) -> +3V3
- U2 pad 3: Net-(D1-K) -> VBUS
Other:
- board outline added: 7.5 x 2 mm
