File: showdown_gun_board.kicad_sch (KiCad schematic)
At the start: 30 parts, among them J1 Conn_01x04_Pin, J2 USB4155-03-C_REVA, SW1 SW_SPDT, U1 AMS1117-3.3, U3 STM32F103C8T6, U5 ${SIM.PARAMS}, Y1 16MHz

Commit message: null
Parts:
- removed C1, C2: 22uF, Capacitor_SMD:C_0603_1608Metric, symbol Device:C
- removed C10, C4, C6, C8, C9: 100nF, Capacitor_SMD:C_0603_1608Metric, symbol Device:C
- removed C11: 10nF, Capacitor_SMD:C_0603_1608Metric, symbol Device:C
- removed C12, C13: 1uF, Capacitor_SMD:C_0603_1608Metric, symbol Device:C
- removed C3: 10uF, Capacitor_SMD:C_0603_1608Metric, symbol Device:C
- removed C5, C7: 10pF, Capacitor_SMD:C_0603_1608Metric, symbol Device:C
- removed D1: BPX65, Package_TO_SOT_THT:TO-18-2_Lens, symbol Sensor_Optical:BPX65
- removed D2: LED_RED, LED_SMD:LED_0805_2012Metric, symbol Device:LED
- removed D3: LED, symbol Device:LED
- removed FB1: 120R, Inductor_SMD:L_0603_1608Metric, symbol Device:FerriteBead
- removed J1: Conn_01x04_Pin, Connector_PinHeader_2.54mm:PinHeader_1x04_P2.54mm_Horizontal, symbol Connector:Conn_01x04_Pin
- removed J2: USB4155-03-C_REVA, USB4155-03-C_REVA:GCT_USB4155-03-C_REVA, symbol USB4155-03-C:USB4155-03-C_REVA
- removed R1: 330R, Resistor_SMD:R_0603_1608Metric, symbol Device:R
- removed R3, R5: 1.5K, Resistor_SMD:R_0603_1608Metric, symbol Device:R
- removed R4: 10K, Resistor_SMD:R_0603_1608Metric, symbol Device:R
- removed R6: 5.1K, Resistor_SMD:R_0603_1608Metric, symbol Device:R
- removed R7: 1M, Resistor_SMD:R_0603_1608Metric, symbol Device:R
- removed SW1: SW_SPDT, Button_Switch_THT:SW_E-Switch_EG1271_SPDT, symbol Switch:SW_SPDT
- removed U1: AMS1117-3.3, Package_TO_SOT_SMD:SOT-223-3_TabPin2, symbol Regulator_Linear:AMS1117-3.3
- removed U3: STM32F103C8T6, Package_QFP:LQFP-48_7x7mm_P0.5mm, symbol MCU_ST_STM32F1:STM32F103C8Tx
- removed U5: ${SIM.PARAMS}, symbol Simulation_SPICE:OPAMP
- removed Y1: 16MHz, Crystal:Crystal_SMD_3225-4Pin_3.2x2.5mm, symbol Device:Crystal_GND24
- added C14, C15: 22uF, Capacitor_SMD:C_0603_1608Metric, symbol Device:C
- added C16: 10uF, Capacitor_SMD:C_0603_1608Metric, symbol Device:C
- added C17, C19, C22, C23, C24: 100nF, Capacitor_SMD:C_0603_1608Metric, symbol Device:C
- added C18, C20: 10pF, Capacitor_SMD:C_0603_1608Metric, symbol Device:C
- added C25: 10nF, Capacitor_SMD:C_0603_1608Metric, symbol Device:C
- added C26, C27: 1uF, Capacitor_SMD:C_0603_1608Metric, symbol Device:C
- added D4: LED_RED, LED_SMD:LED_0805_2012Metric, symbol Device:LED
- added FB2: 120R, Inductor_SMD:L_0603_1608Metric, symbol Device:FerriteBead
- added J3: USB_B_Micro, Connector_USB:USB_Micro-AB_Molex_47590-0001, symbol Connector:USB_B_Micro
- added J4: Conn_01x04_Pin, Connector_PinHeader_2.54mm:PinHeader_1x04_P2.54mm_Horizontal, symbol Connector:Conn_01x04_Pin
- added R18, R21: 1.5K, Resistor_SMD:R_0603_1608Metric, symbol Device:R
- added R19: 10K, Resistor_SMD:R_0603_1608Metric, symbol Device:R
- added SW2: SW_SPDT, Button_Switch_THT:SW_Slide-03_Wuerth-WS-SLTV_10x2.5x6.4_P2.54mm, symbol Switch:SW_SPDT
- added U2: AMS1117-3.3, Package_TO_SOT_SMD:SOT-223-3_TabPin2, symbol Regulator_Linear:AMS1117-3.3
- added U6: STM32F103C8T6, Package_QFP:LQFP-48_7x7mm_P0.5mm, symbol MCU_ST_STM32F1:STM32F103C8Tx
- added Y2: 16MHz, Crystal:Crystal_SMD_3225-4Pin_3.2x2.5mm, symbol Device:Crystal_GND24
Connections:
- net +3V3: now also C15.1, C16.1, C19.1, C22.1, C23.1, C24.1, C27.1, D4.2 (A), FB2.2, J4.1 (Pin_1), R21.2, SW2.3 (C), U2.2 (VO), U6.1 (VBAT), U6.24 (VDD), U6.36 (VDD), U6.48 (VDD)
- net +3V3_A: now also C25.1, C26.1, FB2.1, U6.9 (VDDA)
- net BOOT0: now also R19.2, U6.44 (BOOT0)
- net GND: now also C14.2, C15.2, C16.2, C17.2, C18.2, C19.2, C20.2, C22.2, C23.2, C24.2, C25.2, C26.2, C27.2, J3.5 (GND), J4.4 (Pin_4), R18.1, SW2.1 (A), U2.1 (GND), U6.23 (VSS), U6.35 (VSS), U6.47 (VSS), U6.8 (VSSA), Y2.2, Y2.4
- net HSE_IN: now also C18.1, U6.5 (PD0), Y2.1
- net HSE_OUT: now also C20.1, U6.6 (PD1), Y2.3
- net I2C1_SCL_OLED: now also U6.42 (PB6)
- net I2C1_SDA_OLED: now also U6.43 (PB7)
- net NRST: now also C17.1, U6.7 (NRST)
- net PWR_LED_K: now also D4.1 (K), R18.2
- net SWCLK: now also J4.3 (Pin_3), U6.37 (PA14)
- net SWDIO: now also J4.2 (Pin_2), U6.34 (PA13)
- net SW_BOOT0: now also R19.1, SW2.2 (B)
- net USB_D+: now also J3.3 (D+), R21.1, U6.33 (PA12)
- net USB_D-: now also J3.2 (D-), U6.32 (PA11)
- net VBUS: now also C14.1, J3.1 (VBUS), U2.3 (VI)
- net hit_indicator: now also U6.18 (PB0)
- net hit_register: now also U6.10 (PA0)
- no-connect marks 40 -> 26
Other:
- note added: "VBUS from battery (nom. +3V7) min. 22uF inp./outp. caps"
- note added: "showdown - gun_board"
- note removed: "Detection Circuit"
- note removed: "VBUS from smart phone (nom. +5V0 min. 22uF inp./outp. caps"
- note removed: "showdown - detection board"
- title: showdown - detection board -> showdown - gun board
